Commit message: feat: 添加IMU传感器系统插件到Gazebo仿真环境

File: src/zrobot_gz_sim/resources/zrobot/urdf/zrobot.urdf (robot description, URDF)
Before this commit: robot zrobot, 22 links, 21 joints
Links:
- added link imu_link, mass 0.02; visual sphere radius=0.015
- link L_arm_yaw_link: geometry visual mesh filename=package://zrobot_gz_sim/resources/zrobot/meshes/L_arm_yaw_l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
- link L_elbow_pitch_link: geometry visual mesh filename=package://zrobot_gz_sim/resources/zrobot/meshes/L_elbow_pit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
- link L_foot_pitch_link: geometry visual mesh filename=package://zrobot_gz_sim/resources/zrobot/meshes/L_foot_pitc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
- link L_foot_roll_link: geometry collision mesh filename=package://zrobot_gz_sim/resources/zrobot/meshes/L_foot_roll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; visual mesh filename=package://zrobot_gz_sim/resources/zrobot/meshes/L_foot_roll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
- link L_hip_pitch_link: geometry visual mesh filename=package://zrobot_gz_sim/resources/zrobot/meshes/L_hip_pitch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
- link L_hip_roll_link: geometry visual mesh filename=package://zrobot_gz_sim/resources/zrobot/meshes/L_hip_roll_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
- link L_hip_yaw_link: geometry visual mesh filename=package://zrobot_gz_sim/resources/zrobot/meshes/L_hip_yaw_l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
- link L_knee_link: geometry visual mesh filename=package://zrobot_gz_sim/resources/zrobot/meshes/L_knee_link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
- link L_shoulder_pitch_link: geometry visual mesh filename=package://zrobot_gz_sim/resources/zrobot/meshes/L_shoulder_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
- link L_shoulder_roll_link: geometry visual mesh filename=package://zrobot_gz_sim/resources/zrobot/meshes/L_shoulder_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
- link R_arm_yaw_link: geometry visual mesh filename=package://zrobot_gz_sim/resources/zrobot/meshes/R_arm_yaw_l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
- link R_elbow_pitch_link: geometry visual mesh filename=package://zrobot_gz_sim/resources/zrobot/meshes/R_elbow_pit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
- link R_foot_pitch_link: geometry visual mesh filename=package://zrobot_gz_sim/resources/zrobot/meshes/R_foot_pitc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
- link R_foot_roll_link: geometry collision mesh filename=package://zrobot_gz_sim/resources/zrobot/meshes/R_foot_roll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; visual mesh filename=package://zrobot_gz_sim/resources/zrobot/meshes/R_foot_roll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
- link R_hip_pitch_link: geometry visual mesh filename=package://zrobot_gz_sim/resources/zrobot/meshes/R_hip_pitch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
- link R_hip_roll_link: geometry visual mesh filename=package://zrobot_gz_sim/resources/zrobot/meshes/R_hip_roll_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
- link R_hip_yaw_link: geometry visual mesh filename=package://zrobot_gz_sim/resources/zrobot/meshes/R_hip_yaw_l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
- link R_knee_link: geometry visual mesh filename=package://zrobot_gz_sim/resources/zrobot/meshes/R_knee_link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
- link R_shoulder_pitch_link: geometry visual mesh filename=package://zrobot_gz_sim/resources/zrobot/meshes/R_shoulder_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
- link R_shoulder_roll_link: geometry visual mesh filename=package://zrobot_gz_sim/resources/zrobot/meshes/R_shoulder_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
- link base_link: geometry collision box size=0.195 0.36 0.557; visual mesh filename=package://zrobot_gz_sim/resources/zrobot/meshes/base_link.S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
- link chest_head_link: geometry visual mesh filename=package://zrobot_gz_sim/resources/zrobot/meshes/chest_head_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
Joints:
- added joint imu_joint: type fixed, parent base_link, child imu_link, origin xyz=0 0 0 rpy=0 0 0
